Commit message: message

File: description/robot_model copy.urdf (robot description, URDF)
Before this commit: robot deliver_robot, 5 links, 4 joints
Links:
- link base_link: geometry visual box size=0.3 0.52 0.02
- link chassis: geometry visual box size=0.3 0.52 0.02
Joints:
- removed joint base_joint
- added joint base_link_joint: type fixed, parent base_footprint, child base_link, origin xyz=0.0 0.0 0.1 rpy=0 0 0
- added joint chassis_joint: type fixed, parent base_link, child chassis, origin xyz=0 0 0.1 rpy=0 0 0
- joint laser_joint: origin xyz=0 0 0.2 rpy=0 0 -3.141592 -> xyz=0.07 0 0 rpy=0 0 -3.141592
- joint left_wheel_joint: parent base_link -> base_footprint
- joint right_wheel_joint: parent base_link -> base_footprint
