Commit message: message

File: description/robot_model.urdf (robot description, URDF)
Before this commit: robot deliver_robot, 5 links, 4 joints
Joints:
- joint laser_joint: origin xyz=0 0 0.2 -> xyz=0 0 0.2 rpy=0 0 -3.141592

Commit message: message

File: description/robot_model.urdf (robot description, URDF)
Before this commit: robot deliver_robot, 5 links, 4 joints
Links:
- added link base_footprint
Joints:
- added joint base_footprint_joint: type fixed, parent base_footprint, child base_link, origin xyz=0 0 0.025 rpy=0 0 0

Commit message: commenting esp32_serial_node.py debug handler

File: description/robot_model.urdf (robot description, URDF)
Before this commit: robot deliver_robot, 5 links, 4 joints
Links:
- added link imu; visual cylinder length=0.05 radius=0.03
Joints:
- added joint imu_joint: type fixed, parent base_link, child imu, origin xyz=0 0 0.2 rpy=0 0 0
- joint laser_joint: origin xyz=0 0 0.2 rpy=0 0 -3.141592 -> xyz=0 0 0.3 rpy=0 0 -3.141592; parent chassis -> base_link

Commit message: calibrate encoder odometry

File: description/robot_model.urdf (robot description, URDF)
Before this commit: robot deliver_robot, 6 links, 5 joints
Links:
- added link base_footprint
- link base_link: geometry visual box size=0.3 0.52 0.05
Joints:
- added joint base_footprint_joint: type fixed, parent base_footprint, child base_link, origin xyz=0 0 0.0125 rpy=0 0 0
- joint left_wheel_joint: type continuous -> fixed
- joint right_wheel_joint: type continuous -> fixed
