Commit message: modify to fit base_footprint

File: description/robot_model_legacy.urdf (robot description, URDF)
Before this commit: robot deliver_robot, 7 links, 6 joints
Links:
- link base_link: geometry visual box size=0.3 0.52 0.05
- link chassis: geometry visual box size=0.3 0.52 0.05
- link imu: geometry visual cylinder length=0.05 radius=0.03
- link laser: geometry visual cylinder length=0.05 radius=0.03
Joints:
- joint base_footprint_joint: origin xyz=0 0 0.11 rpy=0 0 0 -> xyz=0 0 0.0125 rpy=0 0 0
- joint base_joint: origin xyz=0 0 0.17 rpy=0 0 0 -> xyz=0 0 0.0125 rpy=0 0 0
- joint imu_joint: origin xyz=0 0 0.15 rpy=0 0 0 -> xyz=0 0 0.2 rpy=0 0 0
- joint laser_joint: origin xyz=0 0 0.2 rpy=0 0 -3.141592 -> xyz=0 0 0.3 rpy=0 0 -3.141592
- joint left_wheel_joint: origin xyz=0 -0.26 0.015 rpy=0 0 0 -> xyz=0 0.21 0.0125 rpy=0 0 0
- joint right_wheel_joint: origin xyz=0 0.26 0.0015 rpy=0 0 0 -> xyz=0 -0.21 0.0125 rpy=0 0 0
